Commit message: Converted to Bebop Simulator

File: hector_quadrotor_gazebo/urdf/camTobi.xacro (robot description, xacro)
@@ -9,13 +9,13 @@
     </joint>
     <link name="${name}_link">
-<!--      <inertial>
+      <inertial>
         <mass value="0.001" />
         <origin xyz="0 0 0" rpy="0 0 0" />
         <inertia ixx="0.0001" ixy="0" ixz="0" iyy="0.0001" iyz="0" izz="0.0001" />
       </inertial>
-      <visual>
+<!--      <visual>
         <origin xyz="0 0 0" rpy="0 0 0" />
         <geometry>
-          <box size="0.01 0.01 0.01" />
+          <box size="0.03 0.1 0.05" />
         </geometry>
         <material name="Blue">

File: hector_quadrotor_gazebo/urdf/gimbal.xacro (robot description, xacro)
@@ -11,14 +11,14 @@
     </joint>
     <link name="${name}_gimbal_root_link">
-      <xacro:inertial_sphere_with_pose mass="0.01" diameter="0.03">
+      <xacro:inertial_sphere_with_pose mass="0.00001" diameter="0.03">
         <origin xyz="0.0 0.0 0.0" rpy="0 0 ${M_PI}"/>
       </xacro:inertial_sphere_with_pose>
     </link>
     <link name="${name}_gimbal_pan_link">
-      <xacro:inertial_sphere_with_pose mass="0.01" diameter="0.01">
+      <xacro:inertial_sphere_with_pose mass="0.00001" diameter="0.01">
         <origin xyz="0 0 0" rpy="0 0 0"/>
       </xacro:inertial_sphere_with_pose>
     </link>
-    <joint name="${name}_gimbal_pan_joint" type="revolute">
+    <joint name="${name}_gimbal_pan_joint" type="revolute" >
       <pose>0 0 0 0 0 0</pose>
       <axis xyz="0 0 1" />
@@ -28,6 +28,19 @@
       <joint_properties damping="2.0" friction="2.0"/>
     </joint>
+    <joint name="${name}_gimbal_roll_joint" type="revolute" >
+      <pose>0 0 0 0 0 0</pose>
+      <axis xyz="1 0 0" />
+      <parent link="${name}_gimbal_pan_link"/>
+      <child link="${name}_gimbal_roll_link"/>
+      <limit effort="1" velocity="0.5" lower="-${M_PI}" upper="${M_PI}"/>
+      <joint_properties damping="2.0" friction="2.0"/>
+    </joint>
+    <link name="${name}_gimbal_roll_link">
+      <xacro:inertial_sphere_with_pose mass="0.00001" diameter="0.01">
+        <origin xyz="0 0 0" rpy="0 0 0"/>
+      </xacro:inertial_sphere_with_pose>
+    </link>
     <link name="${name}_gimbal_tilt_link">
-      <xacro:inertial_sphere_with_pose mass="0.01" diameter="0.01">
+      <xacro:inertial_sphere_with_pose mass="0.00001" diameter="0.01">
         <origin xyz="0 0 0" rpy="0 0 0"/>
       </xacro:inertial_sphere_with_pose>
@@ -36,5 +49,5 @@
       <pose>0 0 0 0 0 0</pose>
       <axis xyz="0 1 0" />
-      <parent link="${name}_gimbal_pan_link"/>
+      <parent link="${name}_gimbal_roll_link"/>
       <child link="${name}_gimbal_tilt_link"/>
       <limit effort="1" velocity="0.5" lower="-${M_PI}" upper="${M_PI}"/>
